File: kicad schematic HPE dl360 gen9/HPE dl360 gen9.kicad_sch (KiCad schematic)
At the start: 0 parts

Commit message: Update KiCad schematics; remove autosaves
Remove autogenerated autosave and lock files and update several KiCad schematics and project files. Embeds a large image into the 10 pin front disk backplane connector schematic and updates connector, fan, front-panel IO schematics, and the main HPE dl360 gen9 project/schematic to reflect those changes. Cleans up clutter (deleted #auto_saved_files#, _autosave-* and .lck) and commits the updated schematic assets.
Other:
- company: (none) -> 0rqa - https://github.com/0rqa
